Commit message: added bump sensor

File: g16_description/urdf/p_g16.gazebo.xacro (robot description, xacro)
@@ -7,4 +7,15 @@
     <material>Gazebo/DarkGrey</material>
     <material>Gazebo/${player_color}</material>
+    <sensor name="base_link" type="contact">
+      <update_rate>1000.0</update_rate>
+      <always_on>true</always_on>
+      <contact>
+        <collision>base_footprint_fixed_joint_lump__base_link_collision</collision>
+      </contact>
+      <plugin name="base_link_contact_sensor_plugin" filename="libgazebo_ros_bumper.so">
+        <bumperTopicName>contact</bumperTopicName>
+        <frameName>world</frameName>
+      </plugin>
+    </sensor>
   </gazebo>
   <gazebo reference="wheel_left_link">

Commit message: added drivers, urdf files and game.yaml

File: g16_description/urdf/p_g16.gazebo.xacro (robot description, xacro)
@@ -8,5 +8,5 @@
     <material>Gazebo/${player_color}</material>
     <sensor name="base_link" type="contact">
-      <update_rate>1000.0</update_rate>
+      <update_rate>10.0</update_rate>
       <always_on>true</always_on>
       <contact>
@@ -19,4 +19,18 @@
     </sensor>
   </gazebo>
+ <!--  <gazebo reference="camera_link">
+    <sensor name="camera_link" type="contact">
+      <update_rate>1000.0</update_rate>
+      <always_on>true</always_on>
+      <contact>
+        <collision>base_footprint_fixed_joint_lump__camera_link_collision</collision>
+      </contact>
+      <plugin name="camera_link_contact_sensor_plugin" filename="libgazebo_ros_bumper.so">
+        <bumperTopicName>contact</bumperTopicName>
+        <frameName>world</frameName>
+      </plugin>
+    </sensor>
+  </gazebo>
+ -->
   <gazebo reference="wheel_left_link">
     <mu1>0.1</mu1>
@@ -115,9 +129,9 @@
   </gazebo>
   <gazebo reference="base_scan">
-    <material>Gazebo/FlatBlack</material>
+    <material>Gazebo/${player_color}</material>
     <sensor type="ray" name="lds_lfcd_sensor">
       <pose>0 0 0 0 0 0</pose>
       <visualize>$(arg laser_visual)</visualize>
-      <update_rate>5</update_rate>
+      <update_rate>10.0</update_rate>
       <ray>
         <scan>
@@ -152,5 +166,5 @@
       <visualize>$(arg camera_visual)</visualize>
       <camera>
-          <horizontal_fov>1.4</horizontal_fov>
+          <horizontal_fov>1.35</horizontal_fov>
           <vertical_fov>1.0</vertical_fov>
           <image>
@@ -166,5 +180,5 @@
       <plugin name="camera_controller" filename="libgazebo_ros_camera.so">
         <alwaysOn>true</alwaysOn>
-        <updateRate>30.0</updateRate>
+        <updateRate>10.0</updateRate>
         <cameraName>camera</cameraName>
         <frameName>camera_rgb_optical_frame</frameName>

File: g16_description/urdf/p_g16.urdf.xacro (robot description, xacro)
@@ -172,10 +172,10 @@
   </joint>
   <link name="camera_link">
-    <collision>
+    <!-- <collision>
       <origin xyz="0.005 0.011 0.013" rpy="0 0 0"/>
       <geometry>
         <box size="0.015 0.030 0.027"/>
       </geometry>
-    </collision>
+    </collision> -->
   </link>
   <joint name="camera_rgb_joint" type="fixed">
